File: pcbs/analog-audio/analog-audio.kicad_pcb (KiCad board)
At the start: 2 copper layers, 83.1 x 70.5 mm, 37 parts, among them J1 AudioJack5, J2 PWR, J5 BASS, J6 TREBLE, J7 Channel, Q1 TIP31, Q2 TIP31, Q3 TIP32, Q4 TIP32, Q5 TIP32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

Commit message: re-designed for power
Parts:
- added R19: 10k, Resistor_THT:R_Axial_DIN0207_L6.3mm_D2.5mm_P7.62mm_Horizontal, F.Cu at (140.0, 118.9)
- added R20: 10k, Resistor_THT:R_Axial_DIN0207_L6.3mm_D2.5mm_P7.62mm_Horizontal, F.Cu at (140.0, 91.4)
- C3, C4: value 10uF -> 1mF; footprint Capacitor_THT:C_Radial_D6.3mm_H11.0mm_P2.50mm -> Capacitor_THT:C_Radial_D10.0mm_H12.5mm_P5.00mm
- J2: value PWR -> 24VDC; footprint TerminalBlock:TerminalBlock_bornier-3_P5.08mm -> Connector_BarrelJack:BarrelJack_GCT_DCJ200-10-A_Horizontal
- moved J2 6.96 mm to (138.2, 109.0), turned to 90 degrees
- moved C4 4.55 mm to (105.5, 107.5)
- moved J6 2.11 mm to (144.6, 134.7)
- moved J5 1.90 mm to (144.4, 77.3)
- moved Q1 1.25 mm to (94.7, 98.2)
- moved Q3 1.25 mm to (94.8, 84.3)
- moved Q5 1.25 mm to (94.8, 136.8)
- moved Q6 1.25 mm to (94.8, 123.2)
- moved C3 1.01 mm to (94.0, 107.5)
Connections:
- C3 pad 1: GND -> +12V
- C3 pad 2: -12V -> GND
- C4 pad 1: +12V -> GND
- C4 pad 2: GND -> -12V
- J2 pad 2: GND -> -12V
- J2 pad 3: -12V -> (no net)
Routing:
- net Net-(Q6-E): track 37.8 -> 73.0 mm, vias 2 -> 0
- net -12V: track 220.4 -> 194.3 mm, vias 0 -> 1
- net VLPF_PA: track 69.9 -> 91.3 mm, vias 0 -> 1
- net VHPF_PA: track 49.2 -> 60.7 mm
- net Net-(Q4-E): track 41.5 -> 51.9 mm
- net +12V: track 228.9 -> 221.9 mm, vias 2 -> 0
- net Net-(Q1-E): track 51.4 -> 57.5 mm, vias 0 -> 1
- net Net-(Q5-E): track 28.1 -> 34.1 mm
- net VTREBLE: track 36.3 -> 40.8 mm
- net Net-(U1--): track 20.2 -> 21.1 mm
- net VBASS: track 44.6 -> 45.3 mm
- net GND: vias 4 -> 28
Other:
- board size 83.1 x 70.5 mm -> 85 x 70.5 mm
- board text added: "AUDIO DRIVER REV 1.0 AV&SS"
- board text removed: "+12V"
- board text removed: "-12V"
- board text removed: "G"

Commit message: added volume control
Parts:
- added J3: VOL-T, Connector_JST:JST_EH_B2B-EH-A_1x02_P2.50mm_Vertical, F.Cu at (108.5, 140.6)
- added J4: VOL-B, Connector_JST:JST_EH_B2B-EH-A_1x02_P2.50mm_Vertical, F.Cu at (111.8, 76.8)
- R3, R4: value 1k -> 820E
- R5, R6: value 6.2k -> 10k
Routing:
- net Net-(J3-Pin_2): track 21.1 -> 56.9 mm, vias 0 -> 2
- net Net-(J4-Pin_2): track 20.0 -> 52.8 mm, vias 0 -> 1
- net VLPF_PA: track 91.3 -> 123.4 mm
- net VHPF_PA: track 60.7 -> 76.0 mm
- net GND: vias 28 -> 20

Commit message: clean up schematic
Routing:
- net GND: vias 20 -> 73

Commit message: re-routed
Parts:
- moved J4 49.0 mm to (66.5, 95.5), turned to -90 degrees
- moved J3 47.9 mm to (66.5, 117.5), turned to -90 degrees
- moved R14 7.75 mm to (87.0, 136.5), turned to 180 degrees
- moved R9 7.70 mm to (76.8, 85.8), turned to 180 degrees
- moved R10 7.70 mm to (76.8, 80.9), turned to 180 degrees
- moved R3 7.70 mm to (76.8, 90.2), turned to 180 degrees
- moved R13 7.68 mm to (76.3, 136.5), turned to 180 degrees
- moved R16 7.62 mm to (87.0, 141.5), turned to 180 degrees
- moved R2 3.26 mm to (80.0, 119.0)
- moved U1 3.08 mm to (76.0, 125.4)
- moved C1 2.52 mm to (74.5, 97.5)
- moved R20 2.14 mm to (138.0, 90.7)
- moved R19 1.77 mm to (138.2, 118.7)
- moved C2 1.52 mm to (86.5, 120.0)
Routing:
- net VLPF_PA: track 123.4 -> 70.0 mm, vias 1 -> 0
- net -12V: track 194.3 -> 231.3 mm, vias 1 -> 0
- net Net-(Q6-E): track 73.0 -> 48.7 mm
- net +12V: track 221.9 -> 199.7 mm, vias 0 -> 1
- net Net-(J3-Pin_2): track 56.9 -> 43.9 mm, vias 2 -> 0
- net Net-(Q4-E): track 51.9 -> 41.5 mm
- net Net-(J4-Pin_2): track 52.8 -> 42.8 mm, vias 1 -> 0
- net VHPF: track 16.8 -> 11.6 mm
- net Vs: track 24.5 -> 28.8 mm
- net VLPF: track 17.2 -> 14.6 mm
- net Net-(Q1-E): track 57.5 -> 59.7 mm, vias 1 -> 0
- net VTREBLE: track 40.8 -> 42.8 mm
- net VBASS: track 45.3 -> 43.4 mm
- net VHPF_PA: track 76.0 -> 77.1 mm
- net Net-(Q5-E): vias 1 -> 0
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- added copper zone on B.Cu, net -12V
