File: pcbs/analog-audio/analog-audio.kicad_pcb (KiCad board)
At the start: 2 copper layers, 85 x 70.5 mm, 41 parts, among them J1 AudioJack5, J2 24VDC, J3 VOL-T, J4 VOL-B, J5 BASS, J6 TREBLE, J7 Channel, Q1 TIP31, Q2 TIP31, Q3 TIP32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

Commit message: add mounting holes
Parts:
- added H1: MountingHole_Pad, MountingHole:MountingHole_3.2mm_M3_Pad_Via, F.Cu at (144.1, 94.2)
- added H2: MountingHole_Pad, MountingHole:MountingHole_3.2mm_M3_Pad_Via, F.Cu at (114.3, 106.3)
- added H3: MountingHole_Pad, MountingHole:MountingHole_3.2mm_M3_Pad_Via, F.Cu at (144.0, 122.6)
- J3: value VOL-T -> VOL
- J4: value VOL-B -> VOL
- R3, R4: value 820E -> 820R
Connections:
- C1 pad 1: GND -> 0
- C3 pad 2: GND -> 0
- C4 pad 1: GND -> 0
- J1 pad S: GND -> 0
- J5 pad 2: GND -> 0
- J6 pad 2: GND -> 0
- R19 pad 2: GND -> 0
- R2 pad 2: GND -> 0
- R20 pad 1: GND -> 0
- U1 pad 3: GND -> 0
Routing:
- net GND: vias 64 -> 0
- net 0: vias 0 -> 48
- added copper zone on B.Cu, net 0
- added copper zone on F.Cu, net 0
- removed copper zone on B.Cu, net GND
- removed copper zone on F.Cu, net GND

Commit message: silkscreen
Parts:
- J3: value VOL -> VOL-T
- J4: value VOL -> VOL-B
Changed lines of the file:
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@@
 			(drillshape 0)
 			(scaleselection 1)
-			(outputdirectory "gerber/")
+			(outputdirectory "outputs/gerber/")
 		)
 	)
@@
 			)
 		)
-		(property "Value" "VOL"
-			(at -5.75 1.75 -90)
+		(property "Value" "VOL-B"
+			(at -5.75 1.75 270)
 			(unlocked yes)
 			(layer "F.SilkS" knockout)
@@
 			)
 		)
-		(property "Value" "VOL"
-			(at 8.25 1.75 -90)
+		(property "Value" "VOL-T"
+			(at 8.25 1.75 270)
 			(unlocked yes)
 			(layer "F.SilkS" knockout)

Commit message: fixed error in PCB and updated to use real values
Parts:
- J4: value VOL-B -> VOL-T
- R10, R15, R16, R8: value 400R -> 1k
- R11, R12: value 1R -> 0.5R
- R3, R4: value 820R -> 750R
Connections:
- U2 pad 3: GND -> 0
